File: m2p.sch (KiCad schematic (older format))
At the start: 40 parts, among them IC1 APU1205-HF-3, IC2 SN74AHC1G32DCKR, IC3 SP100-2T, IC4 ADXL375, IC5 ATMEGA328P, P1 CONN_2, P2 CONN_2, P3 CONN_4, P4 CONN_2, Q1 MOSFET_P, Q3 MOSFET_N, U1 ICSP, U2 RGB LED, X2 8M

Commit message: m2p sch looking good
Parts:
- removed P1: CONN_2, symbol CONN_2
- added C1, C2, C8: 100n, 0603, symbol C
- added C12: 2200µ, symbol CP1
- added D2: DIODESCH, SOT-23, symbol DIODESCH
- added IC2: ADuM1201, symbol ADuM1201
- added P2: CONN_4, symbol CONN_4
- added P4: CONN_2, symbol CONN_2
- added Q2: MOSFET_P, SOT-23, symbol MOSFET_P
- added Q4: MOSFET_N, SOT-23, symbol MOSFET_N
- added R10, R12, R16, R18, R4: 10k, 0603, symbol R
- added R14: 5, symbol R
- added R8, R9: 100, 0603, symbol R
- added U1: BAT BOX, symbol PART
- added U2: ARM SW, symbol PART
- IC3: renamed from IC2; Farnell (none) -> 1287449
- renumbered C7 to C10, C9 to C11, C8 to C13, C11 to C14, C12 to C15, C13 to C16, C1 to C3, C2 to C4, C3 to C5, C4 to C6, C5 to C7, C6 to C9, IC3 to IC4, IC4 to IC5, IC5 to IC6, P2 to P1, P4 to P3, P3 to P5, R12 to R11, R14 to R13, R16 to R15, R18 to R17, R2 to R19, R4 to R2, R3 to R20, R5 to R21, R6 to R3, R8 to R5, R9 to R6, R20 to R7, U2 to U3, U1 to U4, X2 to X1
Connections:
- net PYRO_F_3 is gone; now on net PYRO_C_2: IC6.25 (PC2)
- net PYRO_F_4 is gone; now on net PYRO_F_2: IC6.26 (PC3)
- net +BATT: now also C12.1, Q2.S, R10.2, R4.1
- net GND: now also C12.2, C2.2, C8.2, IC2.4 (GND1), P4.2 (PM), Q4.S, R10.1, R12.2
- net LED_B: now also IC6.1 (PD3); no longer IC6.30 (PD0)
- net LED_G: now also IC6.2 (PD4); no longer IC6.32 (PD2)
- net LED_R: now also IC6.32 (PD2); no longer IC6.28 (PC5/SCL)
- net PYRO_C_1: now also IC6.23 (PC0); no longer IC6.1 (PD3)
- net PYRO_C_2: now also D2.1 (A), R18.2; no longer IC6.2 (PD4)
- net PYRO_F_1: now also IC6.24 (PC1); no longer IC6.23 (PC0)
- net PYRO_F_2: now also R8.2; no longer IC6.24 (PC1)
- net SEROUT: now also IC2.3 (IN_B)
- net VCC: now also C2.1, C8.1, D2.2 (K), IC2.1 (VDD1), R16.2
- net PYRO_C_3: no longer names the net of IC6.9 (PD5)
- net PYRO_C_4: no longer names the net of IC6.10 (PD6)
- net PYRO_C_5: no longer names the net of IC6.11 (PD7)
- net PYRO_F_5: no longer names the net of IC6.27 (PC4/SDA)
- new net: Q4.G, R12.1, R8.1
- new net: P4.1 (P1), R14.1, R16.1, R18.1
- new net: Q2.D, R14.2
- new net: Q2.G, R4.2, R9.1
- new net: Q4.D, R9.2
- new net: C1.2, IC2.8 (VDD2), P2.1 (P1)
- new net: IC2.7 (IN_A), P2.2 (P2)
- new net: IC2.6 (OUT_B), P2.3 (P3)
- new net: C1.1, IC2.5 (GND2), P2.4 (P4)
- new net SERIN: IC2.2 (OUT_A), IC6.30 (PD0)
- no-connect marks 4 -> 13
Other:
- note added: "PYROTECHNIC CIRCUIT 2"
- note added: "SERIAL IN/OUT"
- note added: "STATUS LED"
- note removed: "STATUS OUTPUTS"
- moved on the sheet: C3, IC4, P5, R19, R2, R20, R21, U3
