File: m2p/pcb/m2p.sch (KiCad schematic (older format))
At the start: 102 parts, among them IC1 APU1205-HF-3, IC2 MS5611-01BA03, IC3 ADuM1201, IC4 ADXL375, IC5 STM32F303C, P1 CONN_2, P2 CONN_2, P3 CONN_4, P4 CONN_2, P5 SWD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

Commit message: update farnell codes
Parts:
- IC5: Farnell (none) -> 2333361
Changed lines of the file:
@@
 F 2 "" H 2750 5800 60  0000 C CNN
 F 3 "" H 2750 5800 60  0000 C CNN
+F 4 "2333361" H 2650 5600 60  0001 C CNN "Farnell"
 	1    2650 5600
 	1    0    0    -1
