File: m2r/pcb/m2r.kicad_pcb (KiCad board)
At the start: 2 copper layers, 50 x 75 mm, 118 parts, among them IC1 ADP3338, IC10 STM32F303C, IC11 ADP3333, IC2 ADP3335, IC3 ADuM1201, IC4 ADuM1201, IC5 ADuM1201, IC6 MTX2, IC7 ADL5324, IC8 MAX-7Q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

Commit message: jog logo slightly
Parts:
- moved G*** 1.70 mm to (139.6, 94.2)
Changed lines of the file:
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@@
   )
   (module m2r:cusf_logo_full (layer B.Cu)
-    (at 139.5 95.9)
+    (at 139.6 94.2)
     (fp_text reference G*** (at 0 0) (layer B.SilkS) hide
       (effects (font (thickness 0.3)) (justify mirror))
