File: m2fc/pcb/m2fc.kicad_pcb (KiCad board)
At the start: 4 copper layers, 100 x 70 mm, 351 parts, among them IC101 ADP3335, IC102 STM32F405VGT, IC103 ADP3335, IC201 AD8226, IC202 AD8656, IC203 AD8541, IC204 AD8226, IC205 AD8656, IC206 AD8541, IC207 AD8226, IC208 AD8656, IC209 AD8541, IC301 ADXL375, IC302 ADXL345, IC303 MS5611-01BA03, IC304 HMC5883L, IC305 L3G4200D, IC401 ADuM5201, IC402 ADuM1201, IC601 AD8495, IC602 AD8656, IC603 AD8495, IC604 AD8656, IC605 AD8495, IC606 AD8656, P101 CONN_2, P102 CONN_2, P103 CONN_2, P104 SWD, P201 CONN_4, P202 CONN_4, P203 CONN_4, P401 CONN_4, P402 CONN_2, P403 CONN_4, P501 CONN_2, P502 CONN_2, P503 CONN_2, P601 CONN_2, P602 CONN_2, P603 CONN_2, Q501 MOSFET_P, Q502 MOSFET_N, Q503 MOSFET_P, Q504 MOSFET_N, Q505 MOSFET_P, Q506 MOSFET_N, U106 MICROSD, U107 MOUNT, U108 MOUNT, U109 MOUNT, U110 MOUNT, U111 MOUNT, U112 MOUNT, U113 LOGO, U114 LOGO, X101 8M

Commit message: final checks, tweaks, etc
Parts:
- moved C212 3.00 mm to (64.2, 73.6), turned to 90 degrees
- moved C225 3.00 mm to (75.2, 73.6), turned to 90 degrees
- moved C238 3.00 mm to (86.2, 73.6), turned to 90 degrees
- moved C239 1.40 mm to (84.8, 73.5), turned to 180 degrees
- moved C213 1.40 mm to (62.8, 73.6), turned to 180 degrees
- moved C226 1.40 mm to (73.8, 73.6), turned to 180 degrees
Connections:
- IC102 pad 51: Net-(IC102-Pad51) -> /IMU/LG_ACCEL_CS
- IC202 pad 4: VAA -> GND
- IC202 pad 8: GND -> VAA
- IC205 pad 4: VAA -> GND
- IC205 pad 8: GND -> VAA
- IC208 pad 4: VAA -> GND
- IC208 pad 8: GND -> VAA
- IC602 pad 4: VAA -> GND
- IC602 pad 8: GND -> VAA
- IC604 pad 4: VAA -> GND
- IC604 pad 8: GND -> VAA
- IC606 pad 4: VAA -> GND
- IC606 pad 8: GND -> VAA
Routing:
- net GND: track 553.4 -> 545.1 mm, vias 203 -> 206
- net VAA: track 87.5 -> 92.3 mm, vias 36 -> 33
- net /IMU/LG_ACCEL_CS: track 15.2 -> 19.9 mm
- net Net-(C621-Pad1): track 5.98 -> 6.82 mm
- net Net-(C632-Pad1): track 6.03 -> 6.64 mm
