File: m2fc/pcb/pyros.sch (KiCad schematic (older format))
At the start: 51 parts, among them P501 CONN_2, P502 CONN_2, P503 CONN_2, Q501 MOSFET_P, Q502 MOSFET_N, Q503 MOSFET_P, Q504 MOSFET_N, Q505 MOSFET_P, Q506 MOSFET_N, U501 HOUSING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

Commit message: rescue symbols from m2fc pcb
Parts:
- C501, C502, C503: symbol C -> C-RESCUE-m2fc
- R501, R502, R503, R504, R505, R506, R507, R508, R509, R510, R511, R512, R513, R514, R515, R516, R517, R518, R519, R520, R521: symbol R -> R-RESCUE-m2fc
Changed lines of the file:
@@
 EESchema Schematic File Version 2
+LIBS:m2fc-rescue
 LIBS:power
 LIBS:device
@@
 LIBS:memory
 LIBS:xilinx
-LIBS:special
 LIBS:microcontrollers
 LIBS:dsp
@@
 LIBS:cga0402mlc-12g
 LIBS:m2fc-cache
-EELAYER 24 0
+EELAYER 25 0
 EELAYER END
 $Descr A4 11693 8268
@@
 PYROTECHNIC CIRCUIT 1
 $Comp
-L GND #PWR0155
+L GND-RESCUE-m2fc #PWR0155
 U 1 1 53B98AB3
 P 3650 1750
@@
 $EndComp
 $Comp
-L GND #PWR0156
+L GND-RESCUE-m2fc #PWR0156
 U 1 1 53B98AB9
 P 4600 1950
@@
 $EndComp
 $Comp
-L R R502
+L R-RESCUE-m2fc R502
 U 1 1 53B98ACD
 P 3950 1500
@@
 $EndComp
 $Comp
-L GND #PWR0159
+L GND-RESCUE-m2fc #PWR0159
 U 1 1 53B98AE0
 P 5750 2650
@@
 $EndComp
 $Comp
-L R R505
+L R-RESCUE-m2fc R505
 U 1 1 53B98AE7
 P 5700 2050
@@
 $EndComp
 $Comp
-L R R503
+L R-RESCUE-m2fc R503
 U 1 1 53B98B07
 P 5000 1500
@@
 $EndComp
 $Comp
-L R R507
+L R-RESCUE-m2fc R507
 U 1 1 53B98B0F
 P 5350 2400
@@
 $EndComp
 $Comp
-L R R506
+L R-RESCUE-m2fc R506
 U 1 1 53B98B17
 P 5350 2250
@@
 $EndComp
 $Comp
-L R R501
+L R-RESCUE-m2fc R501
 U 1 1 53B98B1F
 P 5000 1300
@@
 $EndComp
 $Comp
-L R R504
+L R-RESCUE-m2fc R504
 U 1 1 53B98B27
 P 3950 1700
@@
 $EndComp
 $Comp
-L +3.3V #PWR0160
+L +3.3V-RESCUE-m2fc #PWR0160
 U 1 1 53C7F0E7
 P 5050 2200
@@
 $EndComp
 $Comp
-L +3.3V #PWR0161
+L +3.3V-RESCUE-m2fc #PWR0161
 U 1 1 53C7F20C
 P 4800 1900
@@
 $EndComp
 $Comp
-L C C501
+L C-RESCUE-m2fc C501
 U 1 1 53D94B70
 P 4750 2700
@@
 Connection ~ 4900 2400
 $Comp
-L GND #PWR0162
+L GND-RESCUE-m2fc #PWR0162
 U 1 1 53D9528D
 P 4750 2950
@@
 PYROTECHNIC CIRCUIT 2
 $Comp
-L GND #PWR0163
+L GND-RESCUE-m2fc #PWR0163
 U 1 1 53D96F43
 P 3650 3850
@@
 $EndComp
 $Comp
-L GND #PWR0164
+L GND-RESCUE-m2fc #PWR0164
 U 1 1 53D96F49
 P 4600 4050
@@
 $EndComp
 $Comp
-L R R509
+L R-RESCUE-m2fc R509
 U 1 1 53D96F56
 P 3950 3600
@@
 $EndComp
 $Comp
-L GND #PWR0167
+L GND-RESCUE-m2fc #PWR0167
 U 1 1 53D96F62
 P 5750 4750
@@
 $EndComp
 $Comp
-L R R512
+L R-RESCUE-m2fc R512
 U 1 1 53D96F69
 P 5700 4150
@@
 $EndComp
 $Comp
-L R R510
+L R-RESCUE-m2fc R510
 U 1 1 53D96F85
 P 5000 3600
@@
 $EndComp
 $Comp
-L R R514
+L R-RESCUE-m2fc R514
 U 1 1 53D96F8C
 P 5350 4500
@@
 $EndComp
 $Comp
-L R R513
+L R-RESCUE-m2fc R513
 U 1 1 53D96F93
 P 5350 4350
@@
 $EndComp
 $Comp
-L R R508
+L R-RESCUE-m2fc R508
 U 1 1 53D96F9A
 P 5000 3400
@@
 $EndComp
 $Comp
-L R R511
+L R-RESCUE-m2fc R511
 U 1 1 53D96FA1
 P 3950 3800
@@
 $EndComp
 $Comp
-L +3.3V #PWR0168
+L +3.3V-RESCUE-m2fc #PWR0168
 U 1 1 53D96FB6
 P 5050 4300
@@
 $EndComp
 $Comp
-L +3.3V #PWR0169
+L +3.3V-RESCUE-m2fc #PWR0169
 U 1 1 53D96FBC
 P 4800 4000
@@
 $EndComp
 $Comp
-L C C502
+L C-RESCUE-m2fc C502
 U 1 1 53D96FDD
 P 4750 4800
@@
 Connection ~ 4900 4500
 $Comp
-L GND #PWR0170
+L GND-RESCUE-m2fc #PWR0170
 U 1 1 53D97008
 P 4750 5050
@@
 PYROTECHNIC CIRCUIT 3
 $Comp
-L GND #PWR0171
+L GND-RESCUE-m2fc #PWR0171
 U 1 1 53D975FC
 P 3650 5950
@@
 $EndComp
 $Comp
-L GND #PWR0172
+L GND-RESCUE-m2fc #PWR0172
 U 1 1 53D97602
 P 4600 6150
@@
 $EndComp
 $Comp
-L R R516
+L R-RESCUE-m2fc R516
 U 1 1 53D9760F
 P 3950 5700
@@
 $EndComp
 $Comp
-L GND #PWR0175
+L GND-RESCUE-m2fc #PWR0175
 U 1 1 53D9761B
 P 5750 6850
@@
 $EndComp
 $Comp
-L R R519
+L R-RESCUE-m2fc R519
 U 1 1 53D97622
 P 5700 6250
@@
 $EndComp
 $Comp
-L R R517
+L R-RESCUE-m2fc R517
 U 1 1 53D9763E
 P 5000 5700
@@
 $EndComp
 $Comp
-L R R521
+L R-RESCUE-m2fc R521
 U 1 1 53D97645
 P 5350 6600
@@
 $EndComp
 $Comp
-L R R520
+L R-RESCUE-m2fc R520
 U 1 1 53D9764C
 P 5350 6450
@@
 $EndComp
 $Comp
-L R R515
+L R-RESCUE-m2fc R515
 U 1 1 53D97653
 P 5000 5500
@@
 $EndComp
 $Comp
-L R R518
+L R-RESCUE-m2fc R518
 U 1 1 53D9765A
 P 3950 5900
@@
 $EndComp
 $Comp
-L +3.3V #PWR0176
+L +3.3V-RESCUE-m2fc #PWR0176
 U 1 1 53D9766F
 P 5050 6400
@@
 $EndComp
 $Comp
-L +3.3V #PWR0177
+L +3.3V-RESCUE-m2fc #PWR0177
 U 1 1 53D97675
 P 4800 6100
@@
 $EndComp
 $Comp
-L C C503
+L C-RESCUE-m2fc C503
 U 1 1 53D97696
 P 4750 6900
@@
 Connection ~ 4900 6600
 $Comp
-L GND #PWR0178
+L GND-RESCUE-m2fc #PWR0178
 U 1 1 53D976C1
 P 4750 7150
