File: m2fc/pcb/straingauges.sch (KiCad schematic (older format))
At the start: 87 parts, among them IC201 AD8226, IC202 AD8656, IC203 AD8541, IC204 AD8226, IC205 AD8656, IC206 AD8541, IC207 AD8226, IC208 AD8656, IC209 AD8541, P201 CONN_4, P202 CONN_4, P203 CONN_4, U201 HOUSING, U202 HOUSING, U203 HOUSING

Commit message: final checks, tweaks, etc
Connections:
- net GND: now also IC202.4 (V-), IC202.4 (V-), IC205.4 (V-), IC205.4 (V-), IC208.4 (V-), IC208.4 (V-); no longer IC202.8 (V+), IC202.8 (V+), IC205.8 (V+), IC205.8 (V+), IC208.8 (V+), IC208.8 (V+)
- net VAA: now also IC202.8 (V+), IC202.8 (V+), IC205.8 (V+), IC205.8 (V+), IC208.8 (V+), IC208.8 (V+); no longer IC202.4 (V-), IC202.4 (V-), IC205.4 (V-), IC205.4 (V-), IC208.4 (V-), IC208.4 (V-)

Commit message: rescue symbols from m2fc pcb
Parts:
- C201, C202, C203, C204, C205, C206, C207, C208, C209, C210, C211, C212, C213, C214, C215, C216, C217, C218, C219, C220, C221, C222, C223, C224, C225, C226, C227, C228, C229, C230, C231, C232, C233, C234, C235, C236, C237, C238, C239: symbol C -> C-RESCUE-m2fc
- R201, R202, R203, R204, R205, R206, R207, R208, R209, R210, R211, R212, R213, R214, R215, R216, R217, R218, R219, R220, R221, R222, R223, R224: symbol R -> R-RESCUE-m2fc
