File: m2fc/pcb/thermocouples.sch (KiCad schematic (older format))
At the start: 75 parts, among them IC601 AD8495, IC602 AD8656, IC603 AD8495, IC604 AD8656, IC605 AD8495, IC606 AD8656, P601 CONN_2, P602 CONN_2, P603 CONN_2

Commit message: m2fc footprints, start layout
Parts:
- removed C602, C605, C613, C616, C624, C627: 10µ, m2fc:C0603, symbol CP1
- added C602, C605, C613, C616, C624, C627: 10µ, m2fc:C0603, symbol C
- IC602, IC604, IC606: footprint m2fc:SOIC8 -> m2fc:MSOP8; Farnell 1117887 -> 1858055
- R604, R611, R618: Farnell 2117211 -> 2116727
- R605, R612, R619: Farnell 2117373 -> 2116889

Commit message: layout going ok so far...
Connections:
- net GND: now also C611.1, C622.1, C633.1; no longer C611.2, C622.2, C633.2
- net at C608.2, IC601.1 (-IN), R606.1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: now also C611.2; no longer C611.1
- net at C619.2, IC603.1 (-IN), R613.1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: now also C622.2; no longer C622.1
- net at C630.2, IC605.1 (-IN), R620.1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: now also C633.2; no longer C633.1
Changed lines of the file:
@@
 F 4 "2211074" H 1750 2100 60  0001 C CNN "Farnell"
 	1    1750 2100
-	1    0    0    -1
+	-1   0    0    1
 $EndComp
 $Comp
@@
 F 4 "2211074" H 1750 4100 60  0001 C CNN "Farnell"
 	1    1750 4100
-	1    0    0    -1
+	-1   0    0    1
 $EndComp
 $Comp
@@
 F 4 "2211074" H 1750 6100 60  0001 C CNN "Farnell"
 	1    1750 6100
-	1    0    0    -1
-$EndComp
-$Comp
+	-1   0    0    1
+$EndComp
+$Comp

Commit message: paid off woo
Connections:
- net +3.3V renamed VAA

Commit message: final checks, tweaks, etc
Connections:
- net GND: now also IC602.4 (V-), IC602.4 (V-), IC604.4 (V-), IC604.4 (V-), IC606.4 (V-), IC606.4 (V-); no longer IC602.8 (V+), IC602.8 (V+), IC604.8 (V+), IC604.8 (V+), IC606.8 (V+), IC606.8 (V+)
- net VAA: now also IC602.8 (V+), IC602.8 (V+), IC604.8 (V+), IC604.8 (V+), IC606.8 (V+), IC606.8 (V+); no longer IC602.4 (V-), IC602.4 (V-), IC604.4 (V-), IC604.4 (V-), IC606.4 (V-), IC606.4 (V-)

Commit message: rescue symbols from m2fc pcb
Parts:
- C601, C602, C603, C604, C605, C606, C607, C608, C609, C610, C611, C612, C613, C614, C615, C616, C617, C618, C619, C620, C621, C622, C623, C624, C625, C626, C627, C628, C629, C630, C631, C632, C633: symbol C -> C-RESCUE-m2fc
- R601, R602, R603, R604, R605, R606, R607, R608, R609, R610, R611, R612, R613, R614, R615, R616, R617, R618, R619, R620, R621: symbol R -> R-RESCUE-m2fc
