File: m2r/pcb_r2/m2r.kicad_pcb (KiCad board)
At the start: 2 copper layers, 56 x 56 mm, 109 parts, among them IC1 ADP3338, IC10 STM32F303C, IC2 ADP3335, IC3 ADuM1201, IC4 ADuM1201, IC5 ADuM1201, IC6 MTX2, IC8 MAX-7Q, P1 CONN_2, P2 SMA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

Commit message: finished up routing, done silk
Parts:
- removed TP10, TP3, TP5, TP6, TP8, TP9: TESTPAD, m2r:TESTPAD
- added G***: LOGO, m2r:cusf_logo_small, F.Cu at (113.0, 126.5)
- added G***: LOGO, m2r:cusf_logo_full, F.Cu at (102.8, 147.0)
- moved TP17 4.19 mm to (107.5, 155.2)
- moved TP13 2.02 mm to (117.7, 151.5)
- moved Q2 1.10 mm to (93.7, 147.2)
- moved R15 1.10 mm to (92.2, 147.2)
- moved R6 1.10 mm to (92.2, 150.2)
- moved TP28 1.10 mm to (93.7, 145.8)
- moved TP16 0.45 mm to (101.5, 154.1)
- moved P2 0.40 mm to (92.0, 122.6)
- moved P7 0.40 mm to (120.0, 122.6)
- moved D10 0.25 mm to (129.0, 165.2)
- moved D11 0.25 mm to (130.0, 165.2)
Connections:
- IC10 pad 10: (no net) -> Net-(IC10-Pad10)
- IC10 pad 18: (no net) -> Net-(IC10-Pad18)
- IC10 pad 2: (no net) -> Net-(IC10-Pad2)
- IC10 pad 22: (no net) -> Net-(IC10-Pad22)
- IC10 pad 29: (no net) -> Net-(IC10-Pad29)
- IC10 pad 3: (no net) -> Net-(IC10-Pad3)
- IC10 pad 32: (no net) -> Net-(IC10-Pad32)
- IC10 pad 33: (no net) -> Net-(IC10-Pad33)
- IC10 pad 38: (no net) -> Net-(IC10-Pad38)
- IC10 pad 39: (no net) -> Net-(IC10-Pad39)
- IC10 pad 4: (no net) -> Net-(IC10-Pad4)
- IC10 pad 40: (no net) -> Net-(IC10-Pad40)
- IC10 pad 41: (no net) -> Net-(IC10-Pad41)
- IC8 pad 13: (no net) -> Net-(IC8-Pad13)
- IC8 pad 14: (no net) -> Net-(IC8-Pad14)
- IC8 pad 15: (no net) -> Net-(IC8-Pad15)
- IC8 pad 18: (no net) -> Net-(IC8-Pad18)
- IC8 pad 4: (no net) -> Net-(IC8-Pad4)
- IC8 pad 5: (no net) -> Net-(IC8-Pad5)
- P6 pad 6: (no net) -> Net-(P6-Pad6)
- P6 pad 7: (no net) -> Net-(P6-Pad7)
- P6 pad 8: (no net) -> Net-(P6-Pad8)
Routing:
- net GND: track 127.2 -> 277.3 mm, vias 32 -> 94
- net +3V3: track 37.3 -> 172.0 mm, vias 0 -> 10
- net SWDIO: track 12.6 -> 8.18 mm, vias 0 -> 1
- net LED_C: track 50.4 -> 54.7 mm, vias 0 -> 2
- net +BATT: track 23.9 -> 27.2 mm
- net LED_A: track 31.2 -> 33.1 mm, vias 0 -> 2
- net SER_OUT: track 17.0 -> 18.9 mm
- net SER_IN: track 17.1 -> 18.7 mm
- net Net-(IC3-Pad6): track 9.55 -> 8.26 mm
- net Net-(IC4-Pad7): track 9.51 -> 8.34 mm
- net Net-(D10-Pad2): track 17.0 -> 18.2 mm
- net BUZZER: track 9.78 -> 10.8 mm, vias 0 -> 2
- net Net-(C1-Pad1): track 16.7 -> 15.7 mm
- net Net-(IC3-Pad7): track 9.50 -> 8.56 mm
- net Net-(IC4-Pad6): track 9.52 -> 8.64 mm
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Other:
- board text added: "+-"
- board text added: "3v3"
- board text added: "5V"
- board text added: "5v"
- board text added: "6-8VDC IN 5VDC OUT"
- board text added: "ADAM GREIG"
- board text added: "BAT"
- board text added: "LED"
- board text added: "M2FC"
- board text added: "MARTLET 2 RADIO"
- board text added: "RADIO"
- board text added: "RB"
- board text added: "SYS"
- board text added: "cusf.co.uk"
- board text added: "r2 2015-05-23"
- board text removed: "RAD"
- board text removed: "SAT"
- board text removed: "STAT"

Commit message: routing updates
Parts:
- D1, D2: value RED -> GRN
- moved R7 2.20 mm to (109.5, 153.5), turned to 270 degrees
- moved TP27 1.95 mm to (111.0, 156.5)
- moved R9 0.22 mm to (111.0, 153.5), turned to 270 degrees
- moved R8 0.11 mm to (111.0, 150.2), turned to 270 degrees
Connections:
- IC10 pad 29: Net-(IC10-Pad29) -> nRST
Routing:
- net nRST: track 24.1 -> 18.9 mm, vias 1 -> 0
- net Net-(D2-Pad1): track 1.50 -> 3.78 mm
- net SER_IN: track 18.7 -> 20.6 mm, vias 0 -> 2
- net SWCLK: track 14.2 -> 13.1 mm
- net SWDIO: track 8.18 -> 7.33 mm
- net 5V_OUT: track 21.0 -> 20.5 mm
- net +3V3: track 172.0 -> 171.9 mm, vias 10 -> 4
- net SER_OUT: vias 0 -> 2

Commit message: add pinout to bottom silk on m2r-r2
Other:
- board text added: "+"
- board text added: "-"
- board text added: "R"
- board text added: "T"
